File: KiCad/Super_Blaster_v0.1.sch (KiCad schematic (older format))
At the start: 4 parts, among them J2 CONN_02X20, J3 CONN_02X20, J4 CONN_02X20, U2 iCE40-HX8K-CT256

Commit message: top routed?
Parts:
- removed J3, J4: CONN_02X20, Pin_Headers:Pin_Header_Straight_2x20_Pitch1.27mm, symbol CONN_02X20
- removed unit 3 of U2
Connections:
- net labels added: 1.5A_DET, 3A_DET, B3-04_3A, B3-05_3B, B3-06_4A, B3-07_4B, CBSEL_0, CBSEL_1, GPIO0, GPIO1, ~CRESET, ~RESET, ~SIWU
- wire segments 34 -> 72
Other:
- note added: "10"
- note added: "15"
- note added: "17"
- note added: "18"
- moved on the sheet: J2, U2A
Changed lines of the file:
@@
 L iCE40-HX8K-CT256 U2
 U 1 1 58FB0409
-P 4700 2400
-F 0 "U2" H 4900 2650 60  0000 L CNN
-F 1 "iCE40-HX8K-CT256" H 4900 2550 60  0000 L CNN
-F 2 "Homebrew:caBGA_256_.8p_14x14mm" H 4700 2400 60  0001 C CNN
-F 3 "" H 4700 2400 60  0001 C CNN
-	1    4700 2400
+P 3200 3200
+F 0 "U2" H 3400 3450 60  0000 L CNN
+F 1 "iCE40-HX8K-CT256" H 3400 3350 60  0000 L CNN
+F 2 "Homebrew:caBGA_256_.8p_14x14mm" H 3200 3200 60  0001 C CNN
+F 3 "" H 3200 3200 60  0001 C CNN
+	1    3200 3200
 	1    0    0    -1
 $EndComp
@@
 F 3 "" H 7500 1000 60  0001 C CNN
 	2    7500 1000
-	1    0    0    -1
-$EndComp
-$Comp
-L iCE40-HX8K-CT256 U2
-U 3 1 58FB05E6
-P 9000 1000
-F 0 "U2" H 9200 1250 60  0000 L CNN
-F 1 "iCE40-HX8K-CT256" H 9200 1150 60  0000 L CNN
-F 2 "Homebrew:caBGA_256_.8p_14x14mm" H 9000 1000 60  0001 C CNN
-F 3 "" H 9000 1000 60  0001 C CNN
-	3    9000 1000
 	1    0    0    -1
 $EndComp
@@
 F17 "3A_DET" O R 1500 2400 60
 $EndSheet
-Text GLabel 4600 1800 0    60   Input ~ 0
+Text GLabel 1800 3500 0    60   Input ~ 0
 3v3
 $Sheet
@@
 L CONN_02X20 J2
 U 1 1 5911B74C
-P 1850 6550
-F 0 "J2" H 1850 7600 50  0000 C CNN
-F 1 "CONN_02X20" V 1850 6550 50  0000 C CNN
-F 2 "Pin_Headers:Pin_Header_Straight_2x20_Pitch1.27mm" H 1850 5600 50  0001 C CNN
-F 3 "" H 1850 5600 50  0001 C CNN
-	1    1850 6550
-	1    0    0    -1
-$EndComp
-$Comp
-L CONN_02X20 J3
-U 1 1 5911B8B0
-P 3350 4750
-F 0 "J3" H 3350 5800 50  0000 C CNN
-F 1 "CONN_02X20" V 3350 4750 50  0000 C CNN
-F 2 "Pin_Headers:Pin_Header_Straight_2x20_Pitch1.27mm" H 3350 3800 50  0001 C CNN
-F 3 "" H 3350 3800 50  0001 C CNN
-	1    3350 4750
+P 3250 5450
+F 0 "J2" H 3250 6500 50  0000 C CNN
+F 1 "CONN_02X20" V 3250 5450 50  0000 C CNN
+F 2 "Pin_Headers:Pin_Header_Straight_2x20_Pitch1.27mm" H 3250 4500 50  0001 C CNN
+F 3 "" H 3250 4500 50  0001 C CNN
+	1    3250 5450
 	0    -1   -1   0
-$EndComp
-$Comp
-L CONN_02X20 J4
-U 1 1 5911BB24
-P 4750 6550
-F 0 "J4" H 4750 7600 50  0000 C CNN
-F 1 "CONN_02X20" V 4750 6550 50  0000 C CNN
-F 2 "Pin_Headers:Pin_Header_Straight_2x20_Pitch1.27mm" H 4750 5600 50  0001 C CNN
-F 3 "" H 4750 5600 50  0001 C CNN
-	1    4750 6550
-	1    0    0    -1
 $EndComp
 Wire Wire Line
@@
 MEM_SDO
 $Comp
-L Earth #PWR?
+L Earth #PWR01
 U 1 1 59128C7C
-P 4400 2600
-F 0 "#PWR?" H 4400 2350 50  0001 C CNN
-F 1 "Earth" H 4400 2450 50  0001 C CNN
-F 2 "" H 4400 2600 50  0001 C CNN
-F 3 "" H 4400 2600 50  0001 C CNN
-	1    4400 2600
-	1    0    0    -1
-$EndComp
-Wire Wire Line
-	4700 2600 4400 2600
-Wire Wire Line
-	4700 2500 4500 2500
-Wire Wire Line
-	4500 2500 4500 2600
-Connection ~ 4500 2600
-Wire Wire Line
-	4700 2400 4600 2400
-Wire Wire Line
-	4600 2400 4600 2500
-Connection ~ 4600 2500
+P 2900 3400
+F 0 "#PWR01" H 2900 3150 50  0001 C CNN
+F 1 "Earth" H 2900 3250 50  0001 C CNN
+F 2 "" H 2900 3400 50  0001 C CNN
+F 3 "" H 2900 3400 50  0001 C CNN
+	1    2900 3400
+	1    0    0    -1
+$EndComp
+Wire Wire Line
+	2900 3400 3200 3400
+Wire Wire Line
+	3000 3300 3200 3300
+Wire Wire Line
+	3000 3300 3000 3400
+Connection ~ 3000 3400
+Wire Wire Line
+	3200 3200 3100 3200
+Wire Wire Line
+	3100 3200 3100 3300
+Connection ~ 3100 3300
+Wire Wire Line
+	4300 900  3800 900
+Wire Wire Line
+	4300 1000 3800 1000
+Wire Wire Line
+	4300 1100 3800 1100
+Text Label 4300 900  2    60   ~ 0
+~CRESET
+Text Label 4300 1000 2    60   ~ 0
+CBSEL_0
+Text Label 4300 1100 2    60   ~ 0
+CBSEL_1
+Wire Wire Line
+	5500 6000 5900 6000
+Wire Wire Line
+	5500 7300 5000 7300
+Wire Wire Line
+	4000 7300 4500 7300
+Wire Wire Line
+	4500 7400 4000 7400
+Wire Wire Line
+	5500 7400 5000 7400
+Text Label 5500 7300 2    60   ~ 0
+MEM_SS
+Text Label 4000 7300 0    60   ~ 0
+MEM_SCK
+Text Label 4000 7400 0    60   ~ 0
+MEM_SDI
+Text Label 5500 7400 2    60   ~ 0
+MEM_SDO
+Wire Wire Line
+	4500 7500 4400 7500
+Wire Wire Line
+	4400 7500 4400 7600
+Wire Wire Line
+	5000 7500 5100 7500
+Wire Wire Line
+	5100 7500 5100 7600
+$Comp
+L Earth #PWR02
+U 1 1 5913BB93
+P 5100 7600
+F 0 "#PWR02" H 5100 7350 50  0001 C CNN
+F 1 "Earth" H 5100 7450 50  0001 C CNN
+F 2 "" H 5100 7600 50  0001 C CNN
+F 3 "" H 5100 7600 50  0001 C CNN
+	1    5100 7600
+	1    0    0    -1
+$EndComp
+$Comp
+L Earth #PWR03
+U 1 1 5913BF5F
+P 4400 7600
+F 0 "#PWR03" H 4400 7350 50  0001 C CNN
+F 1 "Earth" H 4400 7450 50  0001 C CNN
+F 2 "" H 4400 7600 50  0001 C CNN
+F 3 "" H 4400 7600 50  0001 C CNN
+	1    4400 7600
+	1    0    0    -1
+$EndComp
+Text Notes 2600 2400 0    60   ~ 0
+10
+Text Notes 2600 2300 0    60   ~ 0
+15
+Text Notes 2600 2200 0    60   ~ 0
+18
+Text Notes 2600 2100 0    60   ~ 0
+17
+Text Label 2500 2100 2    60   ~ 0
+GPIO0
+Text Label 2500 2200 2    60   ~ 0
+GPIO1
+Text Label 2500 2300 2    60   ~ 0
+~RESET
+Text Label 2500 2400 2    60   ~ 0
+~SIWU
+Text Label 2500 2500 2    60   ~ 0
+1.5A_DET
+Text Label 2500 2600 2    60   ~ 0
+3A_DET
+Text Label 5500 6000 0    60   ~ 0
+~SIWU
+Text Label 5500 5800 0    60   ~ 0
+~RESET
+Text Label 5500 5600 0    60   ~ 0
+GPIO0
+Text Label 5500 5500 0    60   ~ 0
+GPIO1
+Wire Wire Line
+	5500 5800 5900 5800
+Wire Wire Line
+	5500 5600 5900 5600
+Wire Wire Line
+	5500 5500 5900 5500
+Text Label 5500 6100 0    60   ~ 0
+1.5A_DET
+Text Label 5500 5100 0    60   ~ 0
+3A_DET
+Wire Wire Line
+	5500 5100 5900 5100
+Wire Wire Line
+	5500 6100 5900 6100
+Text GLabel 5800 6400 0    60   Input ~ 0
+3v3
+Wire Wire Line
+	5800 6400 5900 6400
+Wire Wire Line
+	5900 6400 5900 6200
+Wire Wire Line
+	5900 6200 6000 6200
+Wire Wire Line
+	5400 1400 5900 1400
+Wire Wire Line
+	5400 1500 5900 1500
+Wire Wire Line
+	5400 1600 5900 1600
+Wire Wire Line
+	5400 1700 5900 1700
+Wire Wire Line
+	5400 2400 5900 2400
+Wire Wire Line
+	5400 2500 5900 2500
+Wire Wire Line
+	5400 4000 5900 4000
+Wire Wire Line
+	5400 4100 5900 4100
+Wire Wire Line
+	5400 4200 5900 4200
+Wire Wire Line
+	5400 4300 5900 4300
+Wire Wire Line
+	5400 4600 5900 4600
+Wire Wire Line
+	5400 4700 5900 4700
+Wire Wire Line
+	5400 3500 5900 3500
+Wire Wire Line
+	5400 3600 5900 3600
+Wire Wire Line
+	5400 3800 5900 3800
+Wire Wire Line
+	5400 3900 5900 3900
+Wire Wire Line
+	5400 3000 5900 3000
+Wire Wire Line
+	5900 3100 5400 3100
+Text Label 5400 1400 0    60   ~ 0
+B3-04_3A
+Text Label 5400 1500 0    60   ~ 0
+B3-05_3B
+Text Label 5400 1600 0    60   ~ 0
+B3-06_4A
+Text Label 5400 1700 0    60   ~ 0
+B3-07_4B
 $EndSCHEMATC

Commit message: 10_20_2017 update
Parts:
- removed J2: CONN_02X20, Pin_Headers:Pin_Header_Straight_2x20_Pitch1.27mm, symbol CONN_02X20
- added J2, J3, J4: CONN_02X10, Pin_Headers:Pin_Header_Straight_2x10_Pitch1.27mm, symbol CONN_02X10
Connections:
- wire segments 72 -> 78
Other:
- note added: "https://www.digikey.com/product-detail/en/texas-instruments/TXS0108EQPWRQ1/296-42401-1-ND/5356982\n"
Changed lines of the file:
@@
 LIBS:Homebrew
 LIBS:Super_Blaster_v0.1-cache
-EELAYER 25 0
+EELAYER 26 0
 EELAYER END
 $Descr USLetter 11000 8500
@@
 Text Notes 1800 1000 0    60   ~ 0
 Data Bus \nGlobal Pins
-$Comp
-L CONN_02X20 J2
-U 1 1 5911B74C
-P 3250 5450
-F 0 "J2" H 3250 6500 50  0000 C CNN
-F 1 "CONN_02X20" V 3250 5450 50  0000 C CNN
-F 2 "Pin_Headers:Pin_Header_Straight_2x20_Pitch1.27mm" H 3250 4500 50  0001 C CNN
-F 3 "" H 3250 4500 50  0001 C CNN
-	1    3250 5450
-	0    -1   -1   0
-$EndComp
 Wire Wire Line
 	1500 1100 2600 1100
@@
 MEM_SDO
 $Comp
-L Earth #PWR01
+L Earth #PWR1
 U 1 1 59128C7C
 P 2900 3400
-F 0 "#PWR01" H 2900 3150 50  0001 C CNN
+F 0 "#PWR1" H 2900 3150 50  0001 C CNN
 F 1 "Earth" H 2900 3250 50  0001 C CNN
 F 2 "" H 2900 3400 50  0001 C CNN
@@
 	5100 7500 5100 7600
 $Comp
-L Earth #PWR02
+L Earth #PWR3
 U 1 1 5913BB93
 P 5100 7600
-F 0 "#PWR02" H 5100 7350 50  0001 C CNN
+F 0 "#PWR3" H 5100 7350 50  0001 C CNN
 F 1 "Earth" H 5100 7450 50  0001 C CNN
 F 2 "" H 5100 7600 50  0001 C CNN
@@
 $EndComp
 $Comp
-L Earth #PWR03
+L Earth #PWR2
 U 1 1 5913BF5F
 P 4400 7600
-F 0 "#PWR03" H 4400 7350 50  0001 C CNN
+F 0 "#PWR2" H 4400 7350 50  0001 C CNN
 F 1 "Earth" H 4400 7450 50  0001 C CNN
 F 2 "" H 4400 7600 50  0001 C CNN
@@
 Text Label 5400 1700 0    60   ~ 0
 B3-07_4B
+$Comp
+L CONN_02X10 J2
+U 1 1 5959604F
+P 1450 5650
+F 0 "J2" H 1450 6155 15  0000 C CNN
+F 1 "CONN_02X10" V 1450 5650 50  0000 C CNN
+F 2 "Pin_Headers:Pin_Header_Straight_2x10_Pitch1.27mm" H 1450 4450 50  0001 C CNN
+F 3 "" H 1450 4450 50  0001 C CNN
+	1    1450 5650
+	1    0    0    -1
+$EndComp
+$Comp
+L CONN_02X10 J4
+U 1 1 59596F6C
+P 3050 5650
+F 0 "J4" H 3050 6200 50  0000 C CNN
+F 1 "CONN_02X10" V 3050 5650 50  0000 C CNN
+F 2 "Pin_Headers:Pin_Header_Straight_2x10_Pitch1.27mm" H 3050 4450 50  0001 C CNN
+F 3 "" H 3050 4450 50  0001 C CNN
+	1    3050 5650
+	1    0    0    -1
+$EndComp
+$Comp
+L CONN_02X10 J3
+U 1 1 59597077
+P 1450 6950
+F 0 "J3" H 1450 7500 50  0000 C CNN
+F 1 "CONN_02X10" V 1450 6950 50  0000 C CNN
+F 2 "Pin_Headers:Pin_Header_Straight_2x10_Pitch1.27mm" H 1450 5750 50  0001 C CNN
+F 3 "" H 1450 5750 50  0001 C CNN
+	1    1450 6950
+	1    0    0    -1
+$EndComp
+Text Notes 11300 500  0    60   ~ 0
+https://www.digikey.com/product-detail/en/texas-instruments/TXS0108EQPWRQ1/296-42401-1-ND/5356982\n
+$Comp
+L Earth #PWR?
+U 1 1 59EA7DC2
+P 1700 7500
+F 0 "#PWR?" H 1700 7250 50  0001 C CNN
+F 1 "Earth" H 1700 7350 50  0001 C CNN
+F 2 "" H 1700 7500 50  0001 C CNN
+F 3 "" H 1700 7500 50  0001 C CNN
+	1    1700 7500
+	1    0    0    -1
+$EndComp
+$Comp
+L Earth #PWR?
+U 1 1 59EA9876
+P 2800 6200
+F 0 "#PWR?" H 2800 5950 50  0001 C CNN
+F 1 "Earth" H 2800 6050 50  0001 C CNN
+F 2 "" H 2800 6200 50  0001 C CNN
+F 3 "" H 2800 6200 50  0001 C CNN
+	1    2800 6200
+	1    0    0    -1
+$EndComp
+$Comp
+L Earth #PWR?
+U 1 1 59EA9953
+P 1700 6200
+F 0 "#PWR?" H 1700 5950 50  0001 C CNN
+F 1 "Earth" H 1700 6050 50  0001 C CNN
+F 2 "" H 1700 6200 50  0001 C CNN
+F 3 "" H 1700 6200 50  0001 C CNN
+	1    1700 6200
+	1    0    0    -1
+$EndComp
+$Comp
+L Earth #PWR?
+U 1 1 59EAE526
+P 1200 6200
+F 0 "#PWR?" H 1200 5950 50  0001 C CNN
+F 1 "Earth" H 1200 6050 50  0001 C CNN
+F 2 "" H 1200 6200 50  0001 C CNN
+F 3 "" H 1200 6200 50  0001 C CNN
+	1    1200 6200
+	1    0    0    -1
+$EndComp
+$Comp
+L Earth #PWR?
+U 1 1 59EAE6E5
+P 3300 6200
+F 0 "#PWR?" H 3300 5950 50  0001 C CNN
+F 1 "Earth" H 3300 6050 50  0001 C CNN
+F 2 "" H 3300 6200 50  0001 C CNN
+F 3 "" H 3300 6200 50  0001 C CNN
+	1    3300 6200
+	1    0    0    -1
+$EndComp
+$Comp
+L Earth #PWR?
+U 1 1 59EAEB1A
+P 1200 7500
+F 0 "#PWR?" H 1200 7250 50  0001 C CNN
+F 1 "Earth" H 1200 7350 50  0001 C CNN
+F 2 "" H 1200 7500 50  0001 C CNN
+F 3 "" H 1200 7500 50  0001 C CNN
+	1    1200 7500
+	1    0    0    -1
+$EndComp
+Wire Wire Line
+	1700 7400 1700 7500
+Wire Wire Line
+	1200 7400 1200 7500
+Wire Wire Line
+	1700 6100 1700 6200
+Wire Wire Line
+	1200 6100 1200 6200
+Wire Wire Line
+	2800 6100 2800 6200
+Wire Wire Line
+	3300 6100 3300 6200
 $EndSCHEMATC
