File: KiCad/Super_Blaster_v0.1.sch (KiCad schematic (older format))
At the start: 4 parts, among them J2 CONN_02X10, J3 CONN_02X10, J4 CONN_02X10, U2 iCE40-HX8K-CT256

Commit message: 12_11_17 update
Connections:
- net labels added: GND, USB_V
- net labels removed: Earth
- wire segments 78 -> 77
Changed lines of the file:
@@
 LIBS:Homebrew
 LIBS:Super_Blaster_v0.1-cache
-EELAYER 26 0
+EELAYER 25 0
 EELAYER END
 $Descr USLetter 11000 8500
@@
 Text Label 4300 1800 2    60   ~ 0
 MEM_SDO
-$Comp
-L Earth #PWR1
-U 1 1 59128C7C
-P 2900 3400
-F 0 "#PWR1" H 2900 3150 50  0001 C CNN
-F 1 "Earth" H 2900 3250 50  0001 C CNN
-F 2 "" H 2900 3400 50  0001 C CNN
-F 3 "" H 2900 3400 50  0001 C CNN
-	1    2900 3400
-	1    0    0    -1
-$EndComp
 Wire Wire Line
 	2900 3400 3200 3400
 Wire Wire Line
-	3000 3300 3200 3300
-Wire Wire Line
-	3000 3300 3000 3400
-Connection ~ 3000 3400
-Wire Wire Line
 	3200 3200 3100 3200
-Wire Wire Line
-	3100 3200 3100 3300
-Connection ~ 3100 3300
 Wire Wire Line
 	4300 900  3800 900
@@
 Wire Wire Line
 	5100 7500 5100 7600
-$Comp
-L Earth #PWR3
-U 1 1 5913BB93
-P 5100 7600
-F 0 "#PWR3" H 5100 7350 50  0001 C CNN
-F 1 "Earth" H 5100 7450 50  0001 C CNN
-F 2 "" H 5100 7600 50  0001 C CNN
-F 3 "" H 5100 7600 50  0001 C CNN
-	1    5100 7600
-	1    0    0    -1
-$EndComp
-$Comp
-L Earth #PWR2
-U 1 1 5913BF5F
-P 4400 7600
-F 0 "#PWR2" H 4400 7350 50  0001 C CNN
-F 1 "Earth" H 4400 7450 50  0001 C CNN
-F 2 "" H 4400 7600 50  0001 C CNN
-F 3 "" H 4400 7600 50  0001 C CNN
-	1    4400 7600
-	1    0    0    -1
-$EndComp
 Text Notes 2600 2400 0    60   ~ 0
 10
@@
 https://www.digikey.com/product-detail/en/texas-instruments/TXS0108EQPWRQ1/296-42401-1-ND/5356982\n
 $Comp
-L Earth #PWR?
-U 1 1 59EA7DC2
+L GND #PWR01
+U 1 1 5A0FB45B
+P 2900 3400
+F 0 "#PWR01" H 2900 3150 50  0001 C CNN
+F 1 "GND" H 2905 3227 50  0000 C CNN
+F 2 "" H 2900 3400 50  0001 C CNN
+F 3 "" H 2900 3400 50  0001 C CNN
+	1    2900 3400
+	1    0    0    -1
+$EndComp
+$Comp
+L GND #PWR02
+U 1 1 5A0FB611
+P 4400 7600
+F 0 "#PWR02" H 4400 7350 50  0001 C CNN
+F 1 "GND" H 4405 7427 50  0000 C CNN
+F 2 "" H 4400 7600 50  0001 C CNN
+F 3 "" H 4400 7600 50  0001 C CNN
+	1    4400 7600
+	1    0    0    -1
+$EndComp
+$Comp
+L GND #PWR03
+U 1 1 5A0FC05D
+P 5100 7600
+F 0 "#PWR03" H 5100 7350 50  0001 C CNN
+F 1 "GND" H 5105 7427 50  0000 C CNN
+F 2 "" H 5100 7600 50  0001 C CNN
+F 3 "" H 5100 7600 50  0001 C CNN
+	1    5100 7600
+	1    0    0    -1
+$EndComp
+$Comp
+L GND #PWR04
+U 1 1 5A105366
+P 1200 7500
+F 0 "#PWR04" H 1200 7250 50  0001 C CNN
+F 1 "GND" H 1205 7327 50  0000 C CNN
+F 2 "" H 1200 7500 50  0001 C CNN
+F 3 "" H 1200 7500 50  0001 C CNN
+	1    1200 7500
+	1    0    0    -1
+$EndComp
+$Comp
+L GND #PWR05
+U 1 1 5A105AF9
 P 1700 7500
-F 0 "#PWR?" H 1700 7250 50  0001 C CNN
-F 1 "Earth" H 1700 7350 50  0001 C CNN
+F 0 "#PWR05" H 1700 7250 50  0001 C CNN
+F 1 "GND" H 1705 7327 50  0000 C CNN
 F 2 "" H 1700 7500 50  0001 C CNN
 F 3 "" H 1700 7500 50  0001 C CNN
@@
 	1    0    0    -1
 $EndComp
-$Comp
-L Earth #PWR?
-U 1 1 59EA9876
-P 2800 6200
-F 0 "#PWR?" H 2800 5950 50  0001 C CNN
-F 1 "Earth" H 2800 6050 50  0001 C CNN
-F 2 "" H 2800 6200 50  0001 C CNN
-F 3 "" H 2800 6200 50  0001 C CNN
-	1    2800 6200
-	1    0    0    -1
-$EndComp
-$Comp
-L Earth #PWR?
-U 1 1 59EA9953
-P 1700 6200
-F 0 "#PWR?" H 1700 5950 50  0001 C CNN
-F 1 "Earth" H 1700 6050 50  0001 C CNN
-F 2 "" H 1700 6200 50  0001 C CNN
-F 3 "" H 1700 6200 50  0001 C CNN
-	1    1700 6200
-	1    0    0    -1
-$EndComp
-$Comp
-L Earth #PWR?
-U 1 1 59EAE526
-P 1200 6200
-F 0 "#PWR?" H 1200 5950 50  0001 C CNN
-F 1 "Earth" H 1200 6050 50  0001 C CNN
-F 2 "" H 1200 6200 50  0001 C CNN
-F 3 "" H 1200 6200 50  0001 C CNN
-	1    1200 6200
-	1    0    0    -1
-$EndComp
-$Comp
-L Earth #PWR?
-U 1 1 59EAE6E5
-P 3300 6200
-F 0 "#PWR?" H 3300 5950 50  0001 C CNN
-F 1 "Earth" H 3300 6050 50  0001 C CNN
-F 2 "" H 3300 6200 50  0001 C CNN
-F 3 "" H 3300 6200 50  0001 C CNN
-	1    3300 6200
-	1    0    0    -1
-$EndComp
-$Comp
-L Earth #PWR?
-U 1 1 59EAEB1A
-P 1200 7500
-F 0 "#PWR?" H 1200 7250 50  0001 C CNN
-F 1 "Earth" H 1200 7350 50  0001 C CNN
-F 2 "" H 1200 7500 50  0001 C CNN
-F 3 "" H 1200 7500 50  0001 C CNN
-	1    1200 7500
-	1    0    0    -1
-$EndComp
+Wire Wire Line
+	1200 7500 1200 7400
 Wire Wire Line
 	1700 7400 1700 7500
-Wire Wire Line
-	1200 7400 1200 7500
-Wire Wire Line
-	1700 6100 1700 6200
-Wire Wire Line
-	1200 6100 1200 6200
-Wire Wire Line
-	2800 6100 2800 6200
-Wire Wire Line
-	3300 6100 3300 6200
+Text GLabel 1100 7300 0    60   Input ~ 0
+3v3
+Text GLabel 1800 7300 2    60   Input ~ 0
+3v3
+Wire Wire Line
+	1100 7300 1200 7300
+Wire Wire Line
+	1700 7300 1800 7300
+Text GLabel 1800 7200 2    60   Input ~ 0
+USB_V
+Text GLabel 1100 7200 0    60   Input ~ 0
+USB_V
+Wire Wire Line
+	1100 7200 1200 7200
+Wire Wire Line
+	1700 7200 1800 7200
+Wire Wire Line
+	3200 3300 3100 3300
+Wire Wire Line
+	3100 3300 3100 3200
 $EndSCHEMATC

Commit message: switch to beaglepocket outline
Connections:
- no-connect marks 0 -> 2
Changed lines of the file:
@@
 Text Notes 1800 1000 0    60   ~ 0
 Data Bus \nGlobal Pins
-Wire Wire Line
-	1500 1100 2600 1100
-Wire Wire Line
-	1500 1300 2600 1300
-Wire Wire Line
-	1500 1400 2600 1400
-Wire Wire Line
-	2600 1500 1500 1500
-Wire Wire Line
-	1500 1600 2600 1600
-Wire Wire Line
-	2600 1700 1500 1700
-Wire Wire Line
-	1500 1800 2600 1800
-Wire Notes Line
-	1500 900  1800 900
-Wire Notes Line
-	1800 1000 1500 1000
-Wire Notes Line
-	2600 900  2300 900
-Wire Notes Line
-	2600 1000 2300 1000
-Wire Notes Line
-	1500 1200 1800 1200
-Wire Notes Line
-	2200 1200 2600 1200
-Wire Wire Line
-	1500 1900 1800 1900
-Wire Wire Line
-	1500 2000 1800 2000
-Wire Wire Line
-	1500 2100 1800 2100
-Wire Wire Line
-	1500 2200 1800 2200
-Wire Wire Line
-	1500 2300 1800 2300
-Wire Wire Line
-	1800 2400 1500 2400
-Wire Wire Line
-	1800 1900 2000 2100
-Wire Wire Line
-	1800 2000 2000 2200
-Wire Wire Line
-	1800 2100 2000 2300
-Wire Wire Line
-	1800 2200 2000 2400
-Wire Wire Line
-	1800 2300 2000 2500
-Wire Wire Line
-	2000 2600 1800 2400
-Wire Wire Line
-	2000 2100 2500 2100
-Wire Wire Line
-	2000 2200 2500 2200
-Wire Wire Line
-	2000 2300 2500 2300
-Wire Wire Line
-	2000 2400 2500 2400
-Wire Wire Line
-	2000 2500 2500 2500
-Wire Wire Line
-	2000 2600 2500 2600
-Wire Wire Line
-	4300 1500 3800 1500
-Wire Wire Line
-	4300 1600 3800 1600
-Wire Wire Line
-	3800 1700 4300 1700
-Wire Wire Line
-	4300 1800 3800 1800
 Text Label 4300 1500 2    60   ~ 0
 MEM_SS
@@
 Text Label 4300 1800 2    60   ~ 0
 MEM_SDO
-Wire Wire Line
-	2900 3400 3200 3400
-Wire Wire Line
-	3200 3200 3100 3200
-Wire Wire Line
-	4300 900  3800 900
-Wire Wire Line
-	4300 1000 3800 1000
-Wire Wire Line
-	4300 1100 3800 1100
 Text Label 4300 900  2    60   ~ 0
 ~CRESET
@@
 Text Label 4300 1100 2    60   ~ 0
 CBSEL_1
-Wire Wire Line
-	5500 6000 5900 6000
-Wire Wire Line
-	5500 7300 5000 7300
-Wire Wire Line
-	4000 7300 4500 7300
-Wire Wire Line
-	4500 7400 4000 7400
-Wire Wire Line
-	5500 7400 5000 7400
 Text Label 5500 7300 2    60   ~ 0
 MEM_SS
@@
 Text Label 5500 7400 2    60   ~ 0
 MEM_SDO
-Wire Wire Line
-	4500 7500 4400 7500
-Wire Wire Line
-	4400 7500 4400 7600
-Wire Wire Line
-	5000 7500 5100 7500
-Wire Wire Line
-	5100 7500 5100 7600
 Text Notes 2600 2400 0    60   ~ 0
 10
@@
 Text Label 5500 5500 0    60   ~ 0
 GPIO1
-Wire Wire Line
-	5500 5800 5900 5800
-Wire Wire Line
-	5500 5600 5900 5600
-Wire Wire Line
-	5500 5500 5900 5500
 Text Label 5500 6100 0    60   ~ 0
 1.5A_DET
 Text Label 5500 5100 0    60   ~ 0
 3A_DET
-Wire Wire Line
-	5500 5100 5900 5100
-Wire Wire Line
-	5500 6100 5900 6100
 Text GLabel 5800 6400 0    60   Input ~ 0
 3v3
-Wire Wire Line
-	5800 6400 5900 6400
-Wire Wire Line
-	5900 6400 5900 6200
-Wire Wire Line
-	5900 6200 6000 6200
-Wire Wire Line
-	5400 1400 5900 1400
-Wire Wire Line
-	5400 1500 5900 1500
-Wire Wire Line
-	5400 1600 5900 1600
-Wire Wire Line
-	5400 1700 5900 1700
-Wire Wire Line
-	5400 2400 5900 2400
-Wire Wire Line
-	5400 2500 5900 2500
-Wire Wire Line
-	5400 4000 5900 4000
-Wire Wire Line
-	5400 4100 5900 4100
-Wire Wire Line
-	5400 4200 5900 4200
-Wire Wire Line
-	5400 4300 5900 4300
-Wire Wire Line
-	5400 4600 5900 4600
-Wire Wire Line
-	5400 4700 5900 4700
-Wire Wire Line
-	5400 3500 5900 3500
-Wire Wire Line
-	5400 3600 5900 3600
-Wire Wire Line
-	5400 3800 5900 3800
-Wire Wire Line
-	5400 3900 5900 3900
-Wire Wire Line
-	5400 3000 5900 3000
-Wire Wire Line
-	5900 3100 5400 3100
 Text Label 5400 1400 0    60   ~ 0
 B3-04_3A
@@
 L CONN_02X10 J4
 U 1 1 59596F6C
-P 3050 5650
-F 0 "J4" H 3050 6200 50  0000 C CNN
-F 1 "CONN_02X10" V 3050 5650 50  0000 C CNN
-F 2 "Pin_Headers:Pin_Header_Straight_2x10_Pitch1.27mm" H 3050 4450 50  0001 C CNN
-F 3 "" H 3050 4450 50  0001 C CNN
-	1    3050 5650
-	1    0    0    -1
-$EndComp
-$Comp
-L CONN_02X10 J3
-U 1 1 59597077
 P 1450 6950
-F 0 "J3" H 1450 7500 50  0000 C CNN
+F 0 "J4" H 1450 7500 50  0000 C CNN
 F 1 "CONN_02X10" V 1450 6950 50  0000 C CNN
 F 2 "Pin_Headers:Pin_Header_Straight_2x10_Pitch1.27mm" H 1450 5750 50  0001 C CNN
 F 3 "" H 1450 5750 50  0001 C CNN
 	1    1450 6950
+	1    0    0    -1
+$EndComp
+$Comp
+L CONN_02X10 J3
+U 1 1 59597077
+P 3150 5650
+F 0 "J3" H 3150 6200 50  0000 C CNN
+F 1 "CONN_02X10" V 3150 5650 50  0000 C CNN
+F 2 "Pin_Headers:Pin_Header_Straight_2x10_Pitch1.27mm" H 3150 4450 50  0001 C CNN
+F 3 "" H 3150 4450 50  0001 C CNN
+	1    3150 5650
 	1    0    0    -1
 $EndComp
@@
 	1    0    0    -1
 $EndComp
-Wire Wire Line
-	1200 7500 1200 7400
-Wire Wire Line
-	1700 7400 1700 7500
-Text GLabel 1100 7300 0    60   Input ~ 0
+Text GLabel 1100 7200 0    60   Input ~ 0
+3v3
+Text GLabel 1800 7200 2    60   Input ~ 0
 3v3
 Text GLabel 1800 7300 2    60   Input ~ 0
-3v3
+USB_V
+Text GLabel 1100 7300 0    60   Input ~ 0
+USB_V
+Wire Wire Line
+	1500 1100 2600 1100
+Wire Wire Line
+	1500 1300 2600 1300
+Wire Wire Line
+	1500 1400 2600 1400
+Wire Wire Line
+	2600 1500 1500 1500
+Wire Wire Line
+	1500 1600 2600 1600
+Wire Wire Line
+	2600 1700 1500 1700
+Wire Wire Line
+	1500 1800 2600 1800
+Wire Notes Line
+	1500 900  1800 900
+Wire Notes Line
+	1800 1000 1500 1000
+Wire Notes Line
+	2600 900  2300 900
+Wire Notes Line
+	2600 1000 2300 1000
+Wire Notes Line
+	1500 1200 1800 1200
+Wire Notes Line
+	2200 1200 2600 1200
+Wire Wire Line
+	1500 1900 1800 1900
+Wire Wire Line
+	1500 2000 1800 2000
+Wire Wire Line
+	1500 2100 1800 2100
+Wire Wire Line
+	1500 2200 1800 2200
+Wire Wire Line
+	1500 2300 1800 2300
+Wire Wire Line
+	1800 2400 1500 2400
+Wire Wire Line
+	1800 1900 2000 2100
+Wire Wire Line
+	1800 2000 2000 2200
+Wire Wire Line
+	1800 2100 2000 2300
+Wire Wire Line
+	1800 2200 2000 2400
+Wire Wire Line
+	1800 2300 2000 2500
+Wire Wire Line
+	2000 2600 1800 2400
+Wire Wire Line
+	2000 2100 2500 2100
+Wire Wire Line
+	2000 2200 2500 2200
+Wire Wire Line
+	2000 2300 2500 2300
+Wire Wire Line
+	2000 2400 2500 2400
+Wire Wire Line
+	2000 2500 2500 2500
+Wire Wire Line
+	2000 2600 2500 2600
+Wire Wire Line
+	4300 1500 3800 1500
+Wire Wire Line
+	4300 1600 3800 1600
+Wire Wire Line
+	3800 1700 4300 1700
+Wire Wire Line
+	4300 1800 3800 1800
+Wire Wire Line
+	2900 3400 3200 3400
+Wire Wire Line
+	3200 3200 3100 3200
+Wire Wire Line
+	4300 900  3800 900
+Wire Wire Line
+	4300 1000 3800 1000
+Wire Wire Line
+	4300 1100 3800 1100
+Wire Wire Line
+	5500 6000 5900 6000
+Wire Wire Line
+	5500 7300 5000 7300
+Wire Wire Line
+	4000 7300 4500 7300
+Wire Wire Line
+	4500 7400 4000 7400
+Wire Wire Line
+	5500 7400 5000 7400
+Wire Wire Line
+	4500 7500 4400 7500
+Wire Wire Line
+	4400 7500 4400 7600
+Wire Wire Line
+	5000 7500 5100 7500
+Wire Wire Line
+	5100 7500 5100 7600
+Wire Wire Line
+	5500 5800 5900 5800
+Wire Wire Line
+	5500 5600 5900 5600
+Wire Wire Line
+	5500 5500 5900 5500
+Wire Wire Line
+	5500 5100 5900 5100
+Wire Wire Line
+	5500 6100 5900 6100
+Wire Wire Line
+	5800 6400 5900 6400
+Wire Wire Line
+	5900 6400 5900 6200
+Wire Wire Line
+	5900 6200 6000 6200
+Wire Wire Line
+	5400 1400 5900 1400
+Wire Wire Line
+	5400 1500 5900 1500
+Wire Wire Line
+	5400 1600 5900 1600
+Wire Wire Line
+	5400 1700 5900 1700
+Wire Wire Line
+	5400 2400 5900 2400
+Wire Wire Line
+	5400 2500 5900 2500
+Wire Wire Line
+	5400 4000 5900 4000
+Wire Wire Line
+	5400 4100 5900 4100
+Wire Wire Line
+	5400 4200 5900 4200
+Wire Wire Line
+	5400 4300 5900 4300
+Wire Wire Line
+	5400 4600 5900 4600
+Wire Wire Line
+	5400 4700 5900 4700
+Wire Wire Line
+	5400 3500 5900 3500
+Wire Wire Line
+	5400 3600 5900 3600
+Wire Wire Line
+	5400 3800 5900 3800
+Wire Wire Line
+	5400 3900 5900 3900
+Wire Wire Line
+	5400 3000 5900 3000
+Wire Wire Line
+	5900 3100 5400 3100
+Wire Wire Line
+	1200 7500 1200 7400
+Wire Wire Line
+	1700 7400 1700 7500
+Wire Wire Line
+	1100 7200 1200 7200
+Wire Wire Line
+	1700 7200 1800 7200
 Wire Wire Line
 	1100 7300 1200 7300
 Wire Wire Line
 	1700 7300 1800 7300
-Text GLabel 1800 7200 2    60   Input ~ 0
-USB_V
-Text GLabel 1100 7200 0    60   Input ~ 0
-USB_V
-Wire Wire Line
-	1100 7200 1200 7200
-Wire Wire Line
-	1700 7200 1800 7200
 Wire Wire Line
 	3200 3300 3100 3300
 Wire Wire Line
 	3100 3300 3100 3200
+NoConn ~ 3200 4000
+NoConn ~ 3200 3500
 $EndSCHEMATC

Commit message: 4_30_updates
Parts:
- removed J2, J3, J4: CONN_02X10, Pin_Headers:Pin_Header_Straight_2x10_Pitch1.27mm, symbol CONN_02X10
- added C12, C13, C14, C15: 22u, symbol C_Small
- added L1, L2: 2.2u, AdoptedTweaked:L_1008, symbol L_Small
- added R12: 4k7, Resistors_SMD:R_0402, symbol R_Small
- added R13: 9k1, Resistors_SMD:R_0402, symbol R_Small
- added R14: 5k1, Resistors_SMD:R_0402, symbol R_Small
- added R15: 1k6, Resistors_SMD:R_0402, symbol R_Small
- added R16: R_Small, symbol R_Small
- added U5, U6: REG_EN_GND_LX_VIN_NC_FB, TO_SOT_Packages_SMD:TSOT-23-6, symbol REG_EN_GND_LX_VIN_NC_FB
Connections:
- net labels added: 1v2
- net labels removed: B3-04_3A, B3-05_3B, B3-06_4A, B3-07_4B
- wire segments 77 -> 103

Commit message: 7_6_2018 changes
Parts:
- removed R16: R_Small, symbol R_Small
- added C16: .1u, symbol C_Small
- added C17: 10u, symbol C_Small
- added C18, C19, C20, C21, C22, C23, C24, C25, C38, C39, C40, C41, C42, C43: .1u, Capacitors_SMD:C_0402_NoSilk, symbol C_Small
- added D1: D, symbol D
- added J2, J3: Conn_02x25_Odd_Even, AdoptedTweaked:Pin_Header_Straight_2x25_Pitch1.27mm_tight_SMD, symbol Conn_02x25_Odd_Even
- added R17: 100, symbol R_Small
Connections:
- net labels added: CDONE, VLEFT, VTOP
- net labels removed: 1.5A_DET, 3A_DET, GPIO0, GPIO1, ~RESET, ~SIWU
- wire segments 103 -> 113
Other:
- moved on the sheet: C12, C13, C14, C15, L1, L2, R12, R13, R14, R15

Commit message: updated to v5
Parts:
- C12, C13, C14, C15, C17: footprint (none) -> Capacitors_SMD:C_0603; symbol C_Small -> Super_Blaster_v0.1-rescue:C_Small
- C16: footprint (none) -> Capacitors_SMD:C_0402_NoSilk; symbol C_Small -> Super_Blaster_v0.1-rescue:C_Small
- C18, C19, C20, C21, C22, C23, C24, C25, C38, C39, C40, C41, C42, C43: symbol C_Small -> Super_Blaster_v0.1-rescue:C_Small
- D1: footprint (none) -> Diodes_SMD:D_SOD-323; symbol D -> Super_Blaster_v0.1-rescue:D
- J2, J3: symbol Conn_02x25_Odd_Even -> Super_Blaster_v0.1-rescue:Conn_02x25_Odd_Even
- L1, L2: symbol L_Small -> Super_Blaster_v0.1-rescue:L_Small
- R12, R13, R14, R15: symbol R_Small -> Super_Blaster_v0.1-rescue:R_Small
- R17: footprint (none) -> Resistors_SMD:R_0603; symbol R_Small -> Super_Blaster_v0.1-rescue:R_Small
- U2: symbol iCE40-HX8K-CT256 -> Homebrew:iCE40-HX8K-CT256
- U5, U6: footprint TO_SOT_Packages_SMD:TSOT-23-6 -> Package_TO_SOT_SMD:TSOT-23-6; symbol REG_EN_GND_LX_VIN_NC_FB -> Homebrew:REG_EN_GND_LX_VIN_NC_FB
Connections:
- net labels added: ho
- wire segments 113 -> 156
Other:
- moved on the sheet: C18, C19, C20, C21, C22, C23, C24, C25

Commit message: refreshing memory...
Parts:
- D1: footprint Diodes_SMD:D_SOD-323 -> Diode_SMD:D_0402_1005Metric
- U2: symbol Homebrew:iCE40-HX8K-CT256 -> Super_Blaster_v0.1-rescue:iCE40-HX8K-CT256-Homebrew
- U5, U6: symbol Homebrew:REG_EN_GND_LX_VIN_NC_FB -> Super_Blaster_v0.1-rescue:REG_EN_GND_LX_VIN_NC_FB-Homebrew
Changed lines of the file:
@@
 $EndDescr
 $Comp
-L Homebrew:iCE40-HX8K-CT256 U2
+L Super_Blaster_v0.1-rescue:iCE40-HX8K-CT256-Homebrew U2
 U 1 1 58FB0409
 P 5500 3200
@@
 $EndComp
 $Comp
-L Homebrew:iCE40-HX8K-CT256 U2
+L Super_Blaster_v0.1-rescue:iCE40-HX8K-CT256-Homebrew U2
 U 2 1 58FB0482
 P 9300 900
@@
 $EndComp
 $Comp
-L Homebrew:iCE40-HX8K-CT256 U2
+L Super_Blaster_v0.1-rescue:iCE40-HX8K-CT256-Homebrew U2
 U 5 1 58FB070B
 P 7800 900
@@
 $EndComp
 $Comp
-L Homebrew:REG_EN_GND_LX_VIN_NC_FB U5
+L Super_Blaster_v0.1-rescue:REG_EN_GND_LX_VIN_NC_FB-Homebrew U5
 U 1 1 5ADFC0FF
 P 5100 4900
@@
 1v2
 $Comp
-L Homebrew:REG_EN_GND_LX_VIN_NC_FB U6
+L Super_Blaster_v0.1-rescue:REG_EN_GND_LX_VIN_NC_FB-Homebrew U6
 U 1 1 5AE5403A
 P 5100 5700
@@
 F 0 "D1" H 5400 4150 50  0000 C CNN
 F 1 "D" H 5400 3950 50  0000 C CNN
-F 2 "Diodes_SMD:D_SOD-323" H 5400 4050 50  0001 C CNN
+F 2 "Diode_SMD:D_0402_1005Metric" H 5400 4050 50  0001 C CNN
 F 3 "" H 5400 4050 50  0001 C CNN
 	1    5400 4050
