File: KiCad/USB_Conn.sch (KiCad schematic (older format))
At the start: 22 parts, among them J1 USB_TypeC_AMP_12401610E4#2A, U1 LM324, U3 FUSB340, U4 FT601Q, Y1 30MHz

Commit message: 10_20_2017 update
Parts:
- U1: footprint SMD_Packages:SOIC-14_N -> Homebrew:Homebrew-HV-QFN-16
Connections:
- net SS_RX2+ is gone; now on net SS_RX2_P: U3.8 (SSRX2+)
- net SS_RX2- is gone; now on net SS_RX2_N: U3.9 (SSRX2-)
- net T2_P: now reaches C3.1, U3.13 (SSTX2+)
- net T2_N: now reaches C1.2, U3.14 (SSTX2-)
- net T1_P: now reaches C4.1, U3.15 (SSTX1+)
- net T1_N: now reaches C2.2, U3.16 (SSTX1-)
- net Xi: now reaches C7.2, U4.21 (XI), Y1.1
- net Xo: now reaches C6.1, U4.22 (XO), Y1.2
Other:
- note added: "fix footprint pinout"
Changed lines of the file:
@@
 LIBS:Homebrew
 LIBS:Super_Blaster_v0.1-cache
-EELAYER 25 0
+EELAYER 26 0
 EELAYER END
 $Descr USLetter 11000 8500
@@
 USB_D_P
 $Comp
-L Earth #PWR04
+L Earth #PWR11
 U 1 1 5902166F
 P 2900 2500
-F 0 "#PWR04" H 2900 2250 50  0001 C CNN
+F 0 "#PWR11" H 2900 2250 50  0001 C CNN
 F 1 "Earth" H 2900 2350 50  0001 C CNN
 F 2 "" H 2900 2500 50  0001 C CNN
@@
 $EndComp
 $Comp
-L Earth #PWR05
+L Earth #PWR7
 U 1 1 59021695
 P 1500 2500
-F 0 "#PWR05" H 1500 2250 50  0001 C CNN
+F 0 "#PWR7" H 1500 2250 50  0001 C CNN
 F 1 "Earth" H 1500 2350 50  0001 C CNN
 F 2 "" H 1500 2500 50  0001 C CNN
@@
 $EndComp
 $Comp
-L Earth #PWR06
+L Earth #PWR8
 U 1 1 590216D0
 P 1900 2400
-F 0 "#PWR06" H 1900 2150 50  0001 C CNN
+F 0 "#PWR8" H 1900 2150 50  0001 C CNN
 F 1 "Earth" H 1900 2250 50  0001 C CNN
 F 2 "" H 1900 2400 50  0001 C CNN
@@
 $EndComp
 $Comp
-L Earth #PWR07
+L Earth #PWR15
 U 1 1 590216FD
 P 3500 1200
-F 0 "#PWR07" H 3500 950 50  0001 C CNN
+F 0 "#PWR15" H 3500 950 50  0001 C CNN
 F 1 "Earth" H 3500 1050 50  0001 C CNN
 F 2 "" H 3500 1200 50  0001 C CNN
@@
 $EndComp
 $Comp
-L Earth #PWR08
+L Earth #PWR6
 U 1 1 59021728
 P 1000 1200
-F 0 "#PWR08" H 1000 950 50  0001 C CNN
+F 0 "#PWR6" H 1000 950 50  0001 C CNN
 F 1 "Earth" H 1000 1050 50  0001 C CNN
 F 2 "" H 1000 1200 50  0001 C CNN
@@
 $EndComp
 $Comp
-L Earth #PWR09
+L Earth #PWR12
 U 1 1 59027356
 P 3200 4400
-F 0 "#PWR09" H 3200 4150 50  0001 C CNN
+F 0 "#PWR12" H 3200 4150 50  0001 C CNN
 F 1 "Earth" H 3200 4250 50  0001 C CNN
 F 2 "" H 3200 4400 50  0001 C CNN
@@
 SS_RX2_N
 Text Label 2100 3700 0    60   ~ 0
-SS_RX2-
+SS_RX2_N
 Text Label 1200 2100 0    60   ~ 0
 SS_RX2_P
 Text Label 2100 3600 0    60   ~ 0
-SS_RX2+
+SS_RX2_P
 Text Label 1300 3400 0    60   ~ 0
 SS_TX2_P
@@
 $EndComp
 $Comp
-L Earth #PWR010
+L Earth #PWR25
 U 1 1 59035792
 P 6700 5000
-F 0 "#PWR010" H 6700 4750 50  0001 C CNN
+F 0 "#PWR25" H 6700 4750 50  0001 C CNN
 F 1 "Earth" H 6700 4850 50  0001 C CNN
 F 2 "" H 6700 5000 50  0001 C CNN
@@
 $EndComp
 $Comp
-L Earth #PWR011
+L Earth #PWR5
 U 1 1 59037830
 P 900 1700
-F 0 "#PWR011" H 900 1450 50  0001 C CNN
+F 0 "#PWR5" H 900 1450 50  0001 C CNN
 F 1 "Earth" H 900 1550 50  0001 C CNN
 F 2 "" H 900 1700 50  0001 C CNN
@@
 $EndComp
 $Comp
-L Earth #PWR012
+L Earth #PWR16
 U 1 1 59037850
 P 3600 2000
-F 0 "#PWR012" H 3600 1750 50  0001 C CNN
+F 0 "#PWR16" H 3600 1750 50  0001 C CNN
 F 1 "Earth" H 3600 1850 50  0001 C CNN
 F 2 "" H 3600 2000 50  0001 C CNN
@@
 $EndComp
 $Comp
-L Earth #PWR013
+L Earth #PWR9
 U 1 1 590397EE
 P 1900 6300
-F 0 "#PWR013" H 1900 6050 50  0001 C CNN
+F 0 "#PWR9" H 1900 6050 50  0001 C CNN
 F 1 "Earth" H 1900 6150 50  0001 C CNN
 F 2 "" H 1900 6300 50  0001 C CNN
@@
 3v3
 $Comp
-L Earth #PWR014
+L Earth #PWR10
 U 1 1 5903A88C
 P 1900 7600
-F 0 "#PWR014" H 1900 7350 50  0001 C CNN
+F 0 "#PWR10" H 1900 7350 50  0001 C CNN
 F 1 "Earth" H 1900 7450 50  0001 C CNN
 F 2 "" H 1900 7600 50  0001 C CNN
@@
 $EndComp
 $Comp
-L Earth #PWR015
+L Earth #PWR18
 U 1 1 5903A8D0
 P 3900 7600
-F 0 "#PWR015" H 3900 7350 50  0001 C CNN
+F 0 "#PWR18" H 3900 7350 50  0001 C CNN
 F 1 "Earth" H 3900 7450 50  0001 C CNN
 F 2 "" H 3900 7600 50  0001 C CNN
@@
 $EndComp
 $Comp
-L Earth #PWR016
+L Earth #PWR17
 U 1 1 5903A914
 P 3900 6300
-F 0 "#PWR016" H 3900 6050 50  0001 C CNN
+F 0 "#PWR17" H 3900 6050 50  0001 C CNN
 F 1 "Earth" H 3900 6150 50  0001 C CNN
 F 2 "" H 3900 6300 50  0001 C CNN
@@
 $EndComp
 $Comp
-L Earth #PWR017
+L Earth #PWR13
 U 1 1 5903A958
 P 3300 6300
-F 0 "#PWR017" H 3300 6050 50  0001 C CNN
+F 0 "#PWR13" H 3300 6050 50  0001 C CNN
 F 1 "Earth" H 3300 6150 50  0001 C CNN
 F 2 "" H 3300 6300 50  0001 C CNN
@@
 $EndComp
 $Comp
-L Earth #PWR018
+L Earth #PWR14
 U 1 1 5903A9C2
 P 3300 7600
-F 0 "#PWR018" H 3300 7350 50  0001 C CNN
+F 0 "#PWR14" H 3300 7350 50  0001 C CNN
 F 1 "Earth" H 3300 7450 50  0001 C CNN
 F 2 "" H 3300 7600 50  0001 C CNN
@@
 $EndComp
 $Comp
-L Earth #PWR019
+L Earth #PWR19
 U 1 1 5903B44E
 P 4300 3500
-F 0 "#PWR019" H 4300 3250 50  0001 C CNN
+F 0 "#PWR19" H 4300 3250 50  0001 C CNN
 F 1 "Earth" H 4300 3350 50  0001 C CNN
 F 2 "" H 4300 3500 50  0001 C CNN
@@
 F 0 "U1" H 2000 6200 50  0000 L CNN
 F 1 "LM324" H 2000 5800 50  0000 L CNN
-F 2 "SMD_Packages:SOIC-14_N" H 1950 6100 50  0001 C CNN
+F 2 "Homebrew:Homebrew-HV-QFN-16" H 1950 6100 50  0001 C CNN
 F 3 "" H 2050 6200 50  0001 C CNN
 	1    2000 6000
@@
 3A_DET
 $Comp
-L Earth #PWR020
+L Earth #PWR4
 U 1 1 5906A220
 P 800 7350
-F 0 "#PWR020" H 800 7100 50  0001 C CNN
+F 0 "#PWR4" H 800 7100 50  0001 C CNN
 F 1 "Earth" H 800 7200 50  0001 C CNN
 F 2 "" H 800 7350 50  0001 C CNN
@@
 $EndComp
 $Comp
-L Earth #PWR021
+L Earth #PWR24
 U 1 1 59093826
 P 6500 2700
-F 0 "#PWR021" H 6500 2450 50  0001 C CNN
+F 0 "#PWR24" H 6500 2450 50  0001 C CNN
 F 1 "Earth" H 6500 2550 50  0001 C CNN
 F 2 "" H 6500 2700 50  0001 C CNN
@@
 	6100 4800 6100 4700
 $Comp
-L Earth #PWR022
+L Earth #PWR23
 U 1 1 59095C60
 P 6100 5000
-F 0 "#PWR022" H 6100 4750 50  0001 C CNN
+F 0 "#PWR23" H 6100 4750 50  0001 C CNN
 F 1 "Earth" H 6100 4850 50  0001 C CNN
 F 2 "" H 6100 5000 50  0001 C CNN
@@
 $EndComp
 $Comp
-L Earth #PWR023
+L Earth #PWR20
 U 1 1 590967C5
 P 5100 4700
-F 0 "#PWR023" H 5100 4450 50  0001 C CNN
+F 0 "#PWR20" H 5100 4450 50  0001 C CNN
 F 1 "Earth" H 5100 4550 50  0001 C CNN
 F 2 "" H 5100 4700 50  0001 C CNN
@@
 $EndComp
 $Comp
-L Earth #PWR024
+L Earth #PWR21
 U 1 1 59098F88
 P 5300 4200
-F 0 "#PWR024" H 5300 3950 50  0001 C CNN
+F 0 "#PWR21" H 5300 3950 50  0001 C CNN
 F 1 "Earth" H 5300 4050 50  0001 C CNN
 F 2 "" H 5300 4200 50  0001 C CNN
@@
 $EndComp
 $Comp
-L Earth #PWR025
+L Earth #PWR22
 U 1 1 5909A7CE
 P 6100 4200
-F 0 "#PWR025" H 6100 3950 50  0001 C CNN
+F 0 "#PWR22" H 6100 3950 50  0001 C CNN
 F 1 "Earth" H 6100 4050 50  0001 C CNN
 F 2 "" H 6100 4200 50  0001 C CNN
@@
 Text GLabel 7800 3900 2    60   Input ~ 0
 BE_3
+Text Label 2400 3400 0    60   ~ 0
+T2_P
+Text Label 2400 3500 0    60   ~ 0
+T2_N
+Text Label 2400 3900 0    60   ~ 0
+T1_P
+Text Label 2400 4000 0    60   ~ 0
+T1_N
+Text Label 5650 4000 0    60   ~ 0
+Xo
+Text Label 5950 4100 0    60   ~ 0
+Xi
+Text Notes 1000 4800 0    60   ~ 0
+fix footprint pinout
 $EndSCHEMATC

Commit message: 12_11_17 update
Parts:
- added C10: .1uF, Capacitors_SMD:C_0402, symbol C_Small
- added C11: 1nF, Capacitors_SMD:C_0402, symbol C_Small
- added R11: 1M, Resistors_SMD:R_0402, symbol R_Small
- Y1: footprint Crystals:Crystal_SMD_MicroCrystal_CC1V-T1A-2pin_8.0x3.7mm -> Crystals:Crystal_SMD_2016-4pin_2.0x1.6mm; symbol Crystal_Small -> Crystal_GND24; MPN (none) -> XRCGB30M000F3M00R0
Connections:
- net Earth: now also C10.2, C11.2, R11.1; no longer C5.1, C6.2, C7.1, C8.2, J1.A1 (GND), J1.A12 (GND), J1.B1 (GND), J1.B12 (GND), R1.2, R6.2, R8.2, U3.12 (GND[4]), U3.18 (GND[4]), U3.3 (GND[4]), U3.7 (~OE), U3.PAD (GND[4]), U4.1 (GND[5]), U4.26 (GND), U4.29 (GND), U4.36 (GND), U4.77 (GND)
- net Xi: now also Y1.3; no longer Y1.1
- net Xo: now also C6.2, Y1.1; no longer C6.1, Y1.2
- new net GND: C10.1, C11.1, C5.1, C6.1, C7.1, C8.2, J1.A1 (GND), J1.A12 (GND), J1.B1 (GND), J1.B12 (GND), R1.2, R11.2, R6.2, R8.2, U3.12 (GND[4]), U3.18 (GND[4]), U3.3 (GND[4]), U3.7 (~OE), U3.PAD (GND[4]), U4.1 (GND[5]), U4.26 (GND), U4.29 (GND), U4.36 (GND), U4.77 (GND), Y1.2, Y1.4
Other:
- note added: "Switch to uC F103?"
- moved on the sheet: C5, C6, C7, R7

Commit message: switch to beaglepocket outline
Parts:
- Y1: symbol Crystal_GND24 -> Crystal_GND24-RESCUE-Super_Blaster_v0.1
Connections:
- net Earth: no longer R3.2, R5.2, RN1.3 (R3.1), U1.11 (V-), U1.11 (V-), U1.11 (V-), U1.11 (V-)
- net GND: now also R3.2, R5.2, RN1.3 (R3.1), U1.11 (V-), U1.11 (V-), U1.11 (V-), U1.11 (V-)
Other:
- moved on the sheet: RN1, U1B
