File: KiCad/USB_Conn.sch (KiCad schematic (older format))
At the start: 25 parts, among them J1 USB_TypeC_AMP_12401610E4#2A, U1 LM324, U3 FUSB340, U4 FT601Q, Y1 30MHz

Commit message: 4_30_updates
Changed lines of the file:
@@
 USB_D_P
 $Comp
-L Earth #PWR06
+L Earth #PWR012
 U 1 1 590216D0
 P 1900 2500
-F 0 "#PWR06" H 1900 2250 50  0001 C CNN
+F 0 "#PWR012" H 1900 2250 50  0001 C CNN
 F 1 "Earth" H 1900 2350 50  0001 C CNN
 F 2 "" H 1900 2500 50  0001 C CNN
@@
 Text Label 1500 6100 0    60   ~ 0
 CC1
-Text HLabel 6000 4500 0    60   Input ~ 0
+Text HLabel 6100 4500 0    60   Input ~ 0
 ~Wakeup
 Text HLabel 7600 4600 2    60   Input ~ 0
@@
 $EndComp
 Wire Wire Line
-	6200 4600 6000 4600
+	6200 4600 6100 4600
 Wire Wire Line
 	6100 4800 6100 4700
 Wire Wire Line
-	6000 4500 6200 4500
+	6100 4500 6200 4500
 Wire Wire Line
 	6100 4700 6200 4700
 Wire Wire Line
-	4900 4600 5500 4600
+	4900 4600 5600 4600
 $Comp
 L R_Small R7
@@
 Wire Wire Line
 	5100 4200 5100 4300
-Text HLabel 6000 4600 0    60   Input ~ 0
+Text HLabel 6100 4600 0    60   Input ~ 0
 ~SIWU
 Wire Wire Line
@@
 fix footprint pinout
 $Comp
-L GND #PWR07
+L GND #PWR013
 U 1 1 5A0FD17E
-P 5700 6500
-F 0 "#PWR07" H 5700 6250 50  0001 C CNN
-F 1 "GND" H 5705 6327 50  0000 C CNN
-F 2 "" H 5700 6500 50  0001 C CNN
-F 3 "" H 5700 6500 50  0001 C CNN
-	1    5700 6500
-	1    0    0    -1
-$EndComp
-$Comp
-L GND #PWR08
+P 4900 2900
+F 0 "#PWR013" H 4900 2650 50  0001 C CNN
+F 1 "GND" H 4905 2727 50  0000 C CNN
+F 2 "" H 4900 2900 50  0001 C CNN
+F 3 "" H 4900 2900 50  0001 C CNN
+	1    4900 2900
+	1    0    0    -1
+$EndComp
+$Comp
+L GND #PWR014
 U 1 1 5A0FD49F
 P 5100 4900
-F 0 "#PWR08" H 5100 4650 50  0001 C CNN
+F 0 "#PWR014" H 5100 4650 50  0001 C CNN
 F 1 "GND" H 5105 4727 50  0000 C CNN
 F 2 "" H 5100 4900 50  0001 C CNN
@@
 $EndComp
 $Comp
-L GND #PWR09
+L GND #PWR015
 U 1 1 5A0FD567
 P 6100 5000
-F 0 "#PWR09" H 6100 4750 50  0001 C CNN
+F 0 "#PWR015" H 6100 4750 50  0001 C CNN
 F 1 "GND" H 6105 4827 50  0000 C CNN
 F 2 "" H 6100 5000 50  0001 C CNN
@@
 $EndComp
 $Comp
-L GND #PWR010
+L GND #PWR016
 U 1 1 5A0FDBFC
 P 6700 5000
-F 0 "#PWR010" H 6700 4750 50  0001 C CNN
+F 0 "#PWR016" H 6700 4750 50  0001 C CNN
 F 1 "GND" H 6705 4827 50  0000 C CNN
 F 2 "" H 6700 5000 50  0001 C CNN
@@
 $EndComp
 $Comp
-L GND #PWR011
+L GND #PWR017
 U 1 1 5A0FDDF8
 P 6500 2700
-F 0 "#PWR011" H 6500 2450 50  0001 C CNN
+F 0 "#PWR017" H 6500 2450 50  0001 C CNN
 F 1 "GND" H 6505 2527 50  0000 C CNN
 F 2 "" H 6500 2700 50  0001 C CNN
@@
 $EndComp
 $Comp
-L GND #PWR012
+L GND #PWR018
 U 1 1 5A0FE1B4
 P 3500 1200
-F 0 "#PWR012" H 3500 950 50  0001 C CNN
+F 0 "#PWR018" H 3500 950 50  0001 C CNN
 F 1 "GND" H 3505 1027 50  0000 C CNN
 F 2 "" H 3500 1200 50  0001 C CNN
@@
 $EndComp
 $Comp
-L GND #PWR013
+L GND #PWR019
 U 1 1 5A0FE42C
 P 3600 2000
-F 0 "#PWR013" H 3600 1750 50  0001 C CNN
+F 0 "#PWR019" H 3600 1750 50  0001 C CNN
 F 1 "GND" H 3605 1827 50  0000 C CNN
 F 2 "" H 3600 2000 50  0001 C CNN
@@
 $EndComp
 $Comp
-L GND #PWR014
+L GND #PWR020
 U 1 1 5A0FE46D
 P 1000 1200
-F 0 "#PWR014" H 1000 950 50  0001 C CNN
+F 0 "#PWR020" H 1000 950 50  0001 C CNN
 F 1 "GND" H 1005 1027 50  0000 C CNN
 F 2 "" H 1000 1200 50  0001 C CNN
@@
 $EndComp
 $Comp
-L GND #PWR015
+L GND #PWR021
 U 1 1 5A0FE550
 P 900 1700
-F 0 "#PWR015" H 900 1450 50  0001 C CNN
+F 0 "#PWR021" H 900 1450 50  0001 C CNN
 F 1 "GND" H 905 1527 50  0000 C CNN
 F 2 "" H 900 1700 50  0001 C CNN
@@
 $EndComp
 $Comp
-L GND #PWR016
+L GND #PWR022
 U 1 1 5A0FE591
 P 1200 2500
-F 0 "#PWR016" H 1200 2250 50  0001 C CNN
+F 0 "#PWR022" H 1200 2250 50  0001 C CNN
 F 1 "GND" H 1205 2327 50  0000 C CNN
 F 2 "" H 1200 2500 50  0001 C CNN
@@
 $EndComp
 $Comp
-L GND #PWR017
+L GND #PWR023
 U 1 1 5A0FE917
 P 3300 2500
-F 0 "#PWR017" H 3300 2250 50  0001 C CNN
+F 0 "#PWR023" H 3300 2250 50  0001 C CNN
 F 1 "GND" H 3305 2327 50  0000 C CNN
 F 2 "" H 3300 2500 50  0001 C CNN
@@
 $EndComp
 $Comp
-L GND #PWR018
+L GND #PWR024
 U 1 1 5A0FEA4B
 P 4300 3500
-F 0 "#PWR018" H 4300 3250 50  0001 C CNN
+F 0 "#PWR024" H 4300 3250 50  0001 C CNN
 F 1 "GND" H 4305 3327 50  0000 C CNN
 F 2 "" H 4300 3500 50  0001 C CNN
@@
 $EndComp
 $Comp
-L GND #PWR019
+L GND #PWR025
 U 1 1 5A0FEAF8
 P 3200 4400
-F 0 "#PWR019" H 3200 4150 50  0001 C CNN
+F 0 "#PWR025" H 3200 4150 50  0001 C CNN
 F 1 "GND" H 3205 4227 50  0000 C CNN
 F 2 "" H 3200 4400 50  0001 C CNN
@@
 Switch to uC F103?
 $Comp
-L GND #PWR020
+L GND #PWR026
 U 1 1 5A1012D9
 P 5100 4000
-F 0 "#PWR020" H 5100 3750 50  0001 C CNN
+F 0 "#PWR026" H 5100 3750 50  0001 C CNN
 F 1 "GND" V 5105 3872 50  0001 R CNN
 F 2 "" H 5100 4000 50  0001 C CNN
@@
 $EndComp
 $Comp
-L GND #PWR021
+L GND #PWR027
 U 1 1 5A0FDC3D
 P 5400 4400
-F 0 "#PWR021" H 5400 4150 50  0001 C CNN
+F 0 "#PWR027" H 5400 4150 50  0001 C CNN
 F 1 "GND" V 5405 4272 50  0001 R CNN
 F 2 "" H 5400 4400 50  0001 C CNN
@@
 USB_V
 $Comp
-L GND #PWR022
+L GND #PWR028
 U 1 1 5A110AF5
 P 1900 2700
-F 0 "#PWR022" H 1900 2450 50  0001 C CNN
+F 0 "#PWR028" H 1900 2450 50  0001 C CNN
 F 1 "GND" H 1905 2527 50  0000 C CNN
 F 2 "" H 1900 2700 50  0001 C CNN
@@
 Connection ~ 2100 2700
 Wire Wire Line
-	5500 4600 5500 4400
-Wire Wire Line
-	5500 4400 6200 4400
+	5600 4600 5600 4400
+Wire Wire Line
+	5600 4400 6200 4400
 Wire Wire Line
 	5400 4100 5400 4200
@@
 	5200 4000 5100 4000
 $Comp
-L GND #PWR023
+L GND #PWR029
 U 1 1 5A2FAD6A
 P 5600 4000
-F 0 "#PWR023" H 5600 3750 50  0001 C CNN
+F 0 "#PWR029" H 5600 3750 50  0001 C CNN
 F 1 "GND" V 5605 3872 50  0001 R CNN
 F 2 "" H 5600 4000 50  0001 C CNN
@@
 Connection ~ 5400 3800
 $Comp
-L GND #PWR024
+L GND #PWR030
 U 1 1 5A30A472
 P 900 7300
-F 0 "#PWR024" H 900 7050 50  0001 C CNN
+F 0 "#PWR030" H 900 7050 50  0001 C CNN
 F 1 "GND" H 905 7127 50  0000 C CNN
 F 2 "" H 900 7300 50  0001 C CNN
@@
 $EndComp
 $Comp
-L GND #PWR025
+L GND #PWR031
 U 1 1 5A30B01D
 P 3300 7600
-F 0 "#PWR025" H 3300 7350 50  0001 C CNN
+F 0 "#PWR031" H 3300 7350 50  0001 C CNN
 F 1 "GND" H 3305 7427 50  0000 C CNN
 F 2 "" H 3300 7600 50  0001 C CNN
@@
 $EndComp
 $Comp
-L GND #PWR026
+L GND #PWR032
 U 1 1 5A30B082
 P 3900 7600
-F 0 "#PWR026" H 3900 7350 50  0001 C CNN
+F 0 "#PWR032" H 3900 7350 50  0001 C CNN
 F 1 "GND" H 3905 7427 50  0000 C CNN
 F 2 "" H 3900 7600 50  0001 C CNN
@@
 $EndComp
 $Comp
-L GND #PWR027
+L GND #PWR033
 U 1 1 5A30B0E7
 P 3900 6300
-F 0 "#PWR027" H 3900 6050 50  0001 C CNN
+F 0 "#PWR033" H 3900 6050 50  0001 C CNN
 F 1 "GND" H 3905 6127 50  0000 C CNN
 F 2 "" H 3900 6300 50  0001 C CNN
@@
 $EndComp
 $Comp
-L GND #PWR028
+L GND #PWR034
 U 1 1 5A30B14C
 P 3300 6300
-F 0 "#PWR028" H 3300 6050 50  0001 C CNN
+F 0 "#PWR034" H 3300 6050 50  0001 C CNN
 F 1 "GND" H 3305 6127 50  0000 C CNN
 F 2 "" H 3300 6300 50  0001 C CNN
@@
 $EndComp
 $Comp
-L GND #PWR029
+L GND #PWR035
 U 1 1 5A30B1B1
 P 1900 6300
-F 0 "#PWR029" H 1900 6050 50  0001 C CNN
+F 0 "#PWR035" H 1900 6050 50  0001 C CNN
 F 1 "GND" H 1905 6127 50  0000 C CNN
 F 2 "" H 1900 6300 50  0001 C CNN
@@
 $EndComp
 $Comp
-L GND #PWR030
+L GND #PWR036
 U 1 1 5A30C124
 P 2000 7500
-F 0 "#PWR030" H 2000 7250 50  0001 C CNN
+F 0 "#PWR036" H 2000 7250 50  0001 C CNN
 F 1 "GND" H 2005 7327 50  0000 C CNN
 F 2 "" H 2000 7500 50  0001 C CNN

Commit message: 7_6_2018 changes
Parts:
- removed RN1: 1M, Resistors_SMD:R_Array_Concave_4x0402, symbol R_Pack04
- added C26, C28: 1uF, Capacitors_SMD:C_0402, symbol C_Small
- added C27, C29: .1uF, Capacitors_SMD:C_0402, symbol C_Small
- added R18, R19: ?, Resistors_SMD:R_0402, symbol R_Small
Connections:
- net labels removed: 5v
- wire segments 166 -> 168
Other:
- note added: "Summing Amplifier\nbuffers active CC's voltage\n"
- note removed: "Summing Amplifier"

Commit message: updated to v5
Parts:
- removed U1: LM324, Homebrew:Homebrew-HV-QFN-16, symbol LM324
- added U1: MCP6L94, SMD_Packages:SSOP-14, symbol Amplifier_Operational:MCP6L94
- C1, C10, C11, C2, C26, C27, C28, C29, C3, C4, C5, C6, C7, C8: symbol C_Small -> Super_Blaster_v0.1-rescue:C_Small
- J1: symbol USB_TypeC_AMP_12401610E4#2A -> Homebrew:USB_TypeC_AMP_12401610E4#2A
- R1, R11, R18, R19, R2, R3, R4, R5, R6, R7, R8: symbol R_Small -> Super_Blaster_v0.1-rescue:R_Small
- U3: symbol FUSB340 -> Homebrew:FUSB340
- U4: symbol FT601Q -> Homebrew:FT601Q
- U4: footprint (none) -> Homebrew:QFN_76_PAD; symbol FT601Q -> Homebrew:FT601Q
- Y1: footprint Crystals:Crystal_SMD_2016-4pin_2.0x1.6mm -> Crystal:Crystal_SMD_2016-4Pin_2.0x1.6mm; symbol Crystal_GND24-RESCUE-Super_Blaster_v0.1 -> Super_Blaster_v0.1-rescue:Crystal_GND24-RESCUE-Super_Blaster_v0.1
Connections:
- wire segments 168 -> 180

Commit message: refreshing memory...
Parts:
- J1: symbol Homebrew:USB_TypeC_AMP_12401610E4#2A -> Super_Blaster_v0.1-rescue:USB_TypeC_AMP_12401610E4#2A-Homebrew
- U3: symbol Homebrew:FUSB340 -> Super_Blaster_v0.1-rescue:FUSB340-Homebrew
- U4: symbol Homebrew:FT601Q -> Super_Blaster_v0.1-rescue:FT601Q-Homebrew
Changed lines of the file:
@@
 $EndDescr
 $Comp
-L Homebrew:USB_TypeC_AMP_12401610E4#2A J1
+L Super_Blaster_v0.1-rescue:USB_TypeC_AMP_12401610E4#2A-Homebrew J1
 U 1 1 590111D1
 P 2200 1600
@@
 USB_D_N
 $Comp
-L Homebrew:FUSB340 U3
+L Super_Blaster_v0.1-rescue:FUSB340-Homebrew U3
 U 1 1 590272CD
 P 3200 3800
@@
 USB Super Speed Switch to select active channels
 $Comp
-L Homebrew:FT601Q U4
+L Super_Blaster_v0.1-rescue:FT601Q-Homebrew U4
 U 2 1 59028949
 P 8500 5200
@@
 $EndComp
 $Comp
-L Homebrew:FT601Q U4
+L Super_Blaster_v0.1-rescue:FT601Q-Homebrew U4
 U 3 1 590299B6
 P 8400 2200
@@
 $EndComp
 $Comp
-L Homebrew:FT601Q U4
+L Super_Blaster_v0.1-rescue:FT601Q-Homebrew U4
 U 1 1 590288D4
 P 6900 4000
