File: KiCad/Super_Blaster_v0.1.kicad_pcb (KiCad board)
At the start: 4 copper layers, 55 x 35 mm, 34 parts, among them J1 USB_TypeC_AMP_12401610E4#2A, M1 CLOCK_EN, U1 LM324, U2 iCE40-HX8K-CT256, U3 FUSB340, U4 FT601Q, Y1 30MHz

Commit message: 4_30_updates
Parts:
- added L1: 2.2u, AdoptedTweaked:L_1008, F.Cu at (131.0, 97.2)
- added L2: 2.2u, AdoptedTweaked:L_1008, F.Cu at (139.8, 97.2)
- added R12: 4k7, Resistors_SMD:R_0402, F.Cu at (125.4, 94.4)
- added R13: 9k1, Resistors_SMD:R_0402, F.Cu at (125.4, 96.0)
- added R14: 5k1, Resistors_SMD:R_0402, F.Cu at (134.3, 94.3)
- added R15: 1k6, Resistors_SMD:R_0402, F.Cu at (134.3, 95.9)
- added REF**: Pin_Header_Straight_2x30_Pitch1.27mm_SMD, Pin_Headers:Pin_Header_Straight_2x30_Pitch1.27mm_SMD, F.Cu at (149.2, 118.8)
- added U5: REG_EN_GND_LX_VIN_NC_FB, TO_SOT_Packages_SMD:TSOT-23-6, F.Cu at (127.6, 95.9)
- added U6: REG_EN_GND_LX_VIN_NC_FB, TO_SOT_Packages_SMD:TSOT-23-6, F.Cu at (136.5, 95.9)
- moved R10 53.4 mm to (127.6, 83.0)
- moved REF** 23.5 mm to (163.8, 141.4)
- moved RN1 15.2 mm to (116.9, 123.6)
- moved R2 15.2 mm to (119.9, 121.1)
- moved R4 15.2 mm to (112.4, 123.7)
- moved R5 15.2 mm to (112.4, 122.4)
- moved R3 15.2 mm to (118.0, 121.1)
- moved U1 15.2 mm to (120.7, 124.3)
- moved R1 15.2 mm to (114.5, 122.4)
- moved R6 15.2 mm to (114.5, 123.4)
- moved C1 2.51 mm to (129.4, 110.9), turned to 0 degrees
- moved U3 2.47 mm to (134.8, 109.8)
- moved C9 2.35 mm to (144.0, 126.0), turned to 0 degrees
- moved C3 1.65 mm to (129.4, 109.9), turned to 180 degrees
- moved R8 1.65 mm to (138.4, 105.5)
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Connections:
- U2 pad H11: Net-(U2-PadH11) -> /Bottom_Interface/CLK
- U2 pad H16: /Bottom_Interface/CLK -> Net-(U2-PadH16)
- U2 pad J15: D17 -> D16
- U2 pad J16: D16 -> D17
- U2 pad K15: D19 -> D18
- U2 pad K16: D18 -> D19
- U2 pad L14: Net-(U2-PadL14) -> D20
- U2 pad L16: D20 -> D21
- U2 pad M14: Net-(U2-PadM14) -> D24
- U2 pad M16: D21 -> D23
- U2 pad N16: D23 -> D25
- U2 pad P14: Net-(U2-PadP14) -> D28
- U2 pad P15: D24 -> D26
- U2 pad P16: D25 -> D27
- U2 pad R14: Net-(U2-PadR14) -> D31
- U2 pad R15: D26 -> D30
- U2 pad R16: D27 -> D29
- U2 pad T13: D31 -> Net-(U2-PadT13)
- U2 pad T14: D30 -> Net-(U2-PadT14)
- U2 pad T15: D29 -> Net-(U2-PadT15)
- U2 pad T16: D28 -> Net-(U2-PadT16)
Routing:
- net /USB_Connection/SS_RX1_N: track 0.00 -> 19.7 mm, vias 0 -> 2
- net /USB_Connection/SS_RX1_P: track 0.00 -> 18.7 mm, vias 0 -> 2
- net /USB_Connection/T1_N: track 0.00 -> 16.9 mm, vias 0 -> 2
- net /USB_Connection/T1_P: track 0.00 -> 16.9 mm, vias 0 -> 2
- net /USB_Connection/USB_D_N: track 0.00 -> 12.1 mm, vias 0 -> 2
- net /USB_Connection/USB_D_P: track 0.00 -> 11.9 mm
- net /USB_Connection/SS_RX2_N: track 0.00 -> 11.5 mm, vias 0 -> 2
- net /USB_Connection/SS_RX2_P: track 0.00 -> 11.0 mm, vias 0 -> 2
- net /USB_Connection/SS_TX_N: track 0.00 -> 8.09 mm, vias 0 -> 2
- net /USB_Connection/SS_TX_P: track 0.00 -> 8.09 mm, vias 0 -> 2
- net /USB_Connection/SS_RX_N: track 0.00 -> 7.97 mm, vias 0 -> 2
- net /USB_Connection/SS_RX_P: track 0.00 -> 7.97 mm, vias 0 -> 2
- net /USB_Connection/SS_TX2_N: track 0.00 -> 7.83 mm
- net /USB_Connection/SS_TX2_P: track 0.00 -> 7.80 mm
- net Net-(U2-PadH11): track 6.26 -> 0.00 mm, vias 1 -> 0
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Other:
- net class 7mil added: clearance 0.1778, trace_width 0.127, via_dia 0.4572, via_drill 0.254

Commit message: 7_6_2018 changes
Parts:
- removed the REF** at (158.8, 90.8)
- removed the REF** at (163.8, 141.4)
- removed the REF** at (149.2, 118.8)
- added C18: .1u, Capacitors_SMD:C_0402_NoSilk, B.Cu at (161.2, 97.4)
- added C19: .1u, Capacitors_SMD:C_0402_NoSilk, B.Cu at (166.5, 101.6)
- added C20: .1u, Capacitors_SMD:C_0402_NoSilk, B.Cu at (160.1, 103.6)
- added C21: .1u, Capacitors_SMD:C_0402_NoSilk, B.Cu at (161.0, 104.6)
- added C22: .1u, Capacitors_SMD:C_0402_NoSilk, B.Cu at (166.5, 106.2)
- added C23: .1u, Capacitors_SMD:C_0402_NoSilk, B.Cu at (164.7, 109.6)
- added C24: .1u, Capacitors_SMD:C_0402_NoSilk, B.Cu at (161.3, 111.1)
- added C25: .1u, Capacitors_SMD:C_0402_NoSilk, B.Cu at (160.3, 105.7)
- added C26: 1uF, Capacitors_SMD:C_0402, B.Cu at (146.4, 103.6)
- added C27: .1uF, Capacitors_SMD:C_0402, B.Cu at (140.9, 107.8)
- added C28: 1uF, Capacitors_SMD:C_0402, F.Cu at (135.8, 112.6)
- added C29: .1uF, Capacitors_SMD:C_0402, F.Cu at (135.8, 111.9)
- added C30: .1u, Capacitors_SMD:C_0402_NoSilk, B.Cu at (157.9, 98.6)
- added C31: .1u, Capacitors_SMD:C_0402_NoSilk, B.Cu at (152.4, 102.4)
- added C32: .1u, Capacitors_SMD:C_0402_NoSilk, B.Cu at (158.7, 103.9)
- added C33: .1u, Capacitors_SMD:C_0402_NoSilk, B.Cu at (156.3, 100.3)
- added C34: .1u, Capacitors_SMD:C_0402_NoSilk, B.Cu at (158.0, 112.1)
- added C35: .1u, Capacitors_SMD:C_0402_NoSilk, B.Cu at (159.0, 105.3)
- added C36: .1u, Capacitors_SMD:C_0402_NoSilk, B.Cu at (155.1, 107.4)
- added C37: .1u, Capacitors_SMD:C_0402_NoSilk, B.Cu at (153.2, 106.2)
- added C38: .1u, Capacitors_SMD:C_0402_NoSilk, B.Cu at (159.7, 103.2)
- added C39: .1u, Capacitors_SMD:C_0402_NoSilk, B.Cu at (161.4, 105.0)
- added C40: .1u, Capacitors_SMD:C_0402_NoSilk, B.Cu at (161.9, 99.9)
- added C41: .1u, Capacitors_SMD:C_0402_NoSilk, B.Cu at (159.8, 106.2)
- added C42: .1u, Capacitors_SMD:C_0402_NoSilk, B.Cu at (158.2, 104.3)
- added C43: .1u, Capacitors_SMD:C_0402_NoSilk, B.Cu at (160.5, 112.8)
- added C44: .1u, Capacitors_SMD:C_0402_NoSilk, B.Cu at (154.2, 105.6)
- added J2: Conn_02x25_Odd_Even, AdoptedTweaked:Pin_Header_Straight_2x25_Pitch1.27mm_tight_SMD, F.Cu at (150.8, 91.1)
- added J3: Conn_02x25_Odd_Even, AdoptedTweaked:Pin_Header_Straight_2x25_Pitch1.27mm_tight_SMD, F.Cu at (150.8, 119.0)
- added R18: ?, Resistors_SMD:R_0402, F.Cu at (122.4, 113.6)
- added R19: ?, Resistors_SMD:R_0402, F.Cu at (125.0, 112.8)
- D1: value LED_Small -> D; moved to B.Cu
- moved R7 34.5 mm to (143.3, 97.6)
- moved D1 32.2 mm to (159.9, 109.8), turned to 225 degrees
- moved C9 31.9 mm to (152.3, 95.2), turned to 180 degrees
- moved R9 31.5 mm to (139.9, 95.9), turned to 0 degrees
- moved R4 20.3 mm to (131.2, 115.9), turned to 270 degrees
- moved R10 17.3 mm to (139.9, 95.1), turned to 180 degrees
- moved M1 16.9 mm to (152.4, 96.8)
- moved R6 15.7 mm to (127.1, 114.0)
- moved R5 15.4 mm to (125.7, 114.7), turned to 90 degrees
- moved R1 14.9 mm to (127.5, 115.0)
- moved C8 14.0 mm to (140.8, 112.3), turned to 315 degrees
- moved R2 11.0 mm to (129.3, 115.4), turned to 90 degrees
- moved U1 10.5 mm to (129.6, 118.7)
- moved RN1 10.0 mm to (125.3, 118.2), turned to 270 degrees
- moved R3 8.04 mm to (124.3, 116.1), turned to 180 degrees
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Connections:
- net Net-(U2-PadA13) renamed /VTOP
- C5 pad 2: /~RESET -> /Bottom_Interface/~RESET
- D1 pad 1: Earth -> Net-(D1-Pad1)
- D1 pad 2: Net-(D1-Pad2) -> 3v3
- R10 pad 1: 3v3 -> /CDONE
- R10 pad 2: Net-(D1-Pad2) -> 3v3
- R7 pad 2: /~RESET -> /Bottom_Interface/~RESET
- U1 pad 14: /3A_DET -> /Bottom_Interface/3A_DET
- U1 pad 5: Net-(RN1-Pad7) -> Net-(R18-Pad2)
- U1 pad 6: Net-(RN1-Pad5) -> /USB_Connection/CCV
- U1 pad 8: /1.5A_DET -> /Bottom_Interface/1.5A_DET
- U2 pad A14: Net-(U2-PadA14) -> 1v2
- U2 pad D15: D4 -> D5
- U2 pad E1: 3v3 -> /VLEFT
- U2 pad E12: Net-(U2-PadE12) -> Net-(D1-Pad1)
- U2 pad E13: D9 -> D6
- U2 pad E14: D8 -> D4
- U2 pad E16: D5 -> D7
- U2 pad E8: Net-(U2-PadE8) -> Net-(C16-Pad2)
- U2 pad F10: Net-(U2-PadA14) -> 1v2
- U2 pad F13: D11 -> D12
- U2 pad F14: D6 -> D8
- U2 pad F15: D13 -> D11
- U2 pad F16: D7 -> D9
- U2 pad F6: Net-(U2-PadA14) -> 1v2
- U2 pad G12: D12 -> D14
- U2 pad G16: D14 -> D13
- U2 pad G6: 3v3 -> /VLEFT
- U2 pad J6: 3v3 -> /VLEFT
- U2 pad K10: Net-(U2-PadA14) -> 1v2
- U2 pad K6: Net-(U2-PadA14) -> 1v2
- U2 pad L2: Net-(U2-PadA14) -> 1v2
- U2 pad L8: Net-(U2-PadL8) -> Net-(C16-Pad2)
- U2 pad M10: Net-(D1-Pad2) -> /CDONE
- U2 pad N1: 3v3 -> /VLEFT
- U2 pad R10: Net-(U2-PadR10) -> BE_3
- U2 pad R3: Net-(U2-PadR3) -> /Bottom_Interface/GPIO1
- U2 pad R4: Net-(U2-PadR4) -> /Bottom_Interface/GPIO0
- U2 pad R5: Net-(U2-PadR5) -> /Bottom_Interface/~RESET
- U2 pad R6: Net-(U2-PadR6) -> /Bottom_Interface/~RD
- U2 pad T10: Net-(U2-PadT10) -> /Bottom_Interface/~TXE
- U2 pad T11: Net-(U2-PadT11) -> BE_2
- U2 pad T13: Net-(U2-PadT13) -> BE_1
- U2 pad T14: Net-(U2-PadT14) -> BE_0
- U2 pad T15: Net-(U2-PadT15) -> /Bottom_Interface/3A_DET
- U2 pad T16: Net-(U2-PadT16) -> /Bottom_Interface/1.5A_DET
- U2 pad T5: Net-(U2-PadT5) -> /Bottom_Interface/~Wakeup
- U2 pad T6: Net-(U2-PadT6) -> /Bottom_Interface/~OE
- U2 pad T7: Net-(U2-PadT7) -> /Bottom_Interface/~WR
- U2 pad T8: Net-(U2-PadT8) -> /Bottom_Interface/~SIWU
- U2 pad T9: Net-(U2-PadT9) -> /Bottom_Interface/~RXF
- U4 pad 10: /~SIWU -> /Bottom_Interface/~SIWU
- U4 pad 15: /~RESET -> /Bottom_Interface/~RESET
- U4 pad 17: /GPIO0 -> /Bottom_Interface/GPIO0
- U4 pad 18: /GPIO1 -> /Bottom_Interface/GPIO1
- U4 pad 37: 5v -> USB_V
Routing:
- net GND: track 26.4 -> 88.0 mm, vias 15 -> 19
- net /CDONE: track 0.00 -> 28.8 mm, vias 0 -> 3
- net /~CRESET: track 0.00 -> 27.7 mm, vias 0 -> 3
- net /CBSEL_0: track 0.00 -> 26.6 mm, vias 0 -> 2
- net /MEM_SCK: track 2.62 -> 26.4 mm, vias 1 -> 2
- net /MEM_SS: track 4.09 -> 27.0 mm, vias 1 -> 2
- net /Bottom_Interface/GPIO1: track 0.00 -> 21.3 mm
- net /MEM_SDI: track 4.39 -> 25.2 mm, vias 1 -> 2
- net Net-(U2-PadB12): track 0.00 -> 19.9 mm
- net /MEM_SDO: track 5.85 -> 25.5 mm, vias 1 -> 2
- net /Bottom_Interface/GPIO0: track 0.00 -> 19.6 mm
- net /Bottom_Interface/~RESET: track 0.00 -> 18.0 mm
- net /Bottom_Interface/~Wakeup: track 0.00 -> 17.8 mm
- net Net-(U2-PadB14): track 0.00 -> 17.5 mm
- net Net-(U2-PadB13): track 0.00 -> 17.0 mm, vias 0 -> 1
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Other:
- board text removed: "3.3V power"

Commit message: updated to v5
Parts:
- removed REF**: Pin_Header_Straight_2x08_Pitch2.54mm, Pin_Headers:Pin_Header_Straight_2x08_Pitch2.54mm
- removed RN1: 1M, Resistors_SMD:R_Array_Concave_4x0402
- added C12: 22u, Capacitors_SMD:C_0603, F.Cu at (125.9, 96.7)
- added C13: 22u, Capacitors_SMD:C_0603, F.Cu at (125.9, 91.0)
- added C14: 22u, Capacitors_SMD:C_0603, F.Cu at (133.3, 92.9)
- added C15: 22u, Capacitors_SMD:C_0603, F.Cu at (133.4, 98.9)
- added C16: .1u, Capacitors_SMD:C_0402_NoSilk, B.Cu at (162.6, 106.1)
- added C17: 10u, Capacitors_SMD:C_0603, B.Cu at (158.3, 101.9)
- added R17: 100, Resistors_SMD:R_0603, B.Cu at (160.9, 107.2)
- D1: footprint LEDs:LED_0603 -> Diodes_SMD:D_SOD-323
- M1: footprint Crystals:Crystal_SMD_2520-4pin_2.5x2.0mm -> Crystal:Crystal_SMD_2520-4Pin_2.5x2.0mm
- R1, R6: moved to B.Cu
- U1: value LM324 -> MCP6L94; footprint Homebrew:Homebrew-HV-QFN-16 -> SMD_Packages:SSOP-14
- U5, U6: footprint TO_SOT_Packages_SMD:TSOT-23-6 -> Package_TO_SOT_SMD:TSOT-23-6
- Y1: footprint Crystals:Crystal_SMD_2016-4pin_2.0x1.6mm -> Crystal:Crystal_SMD_2016-4Pin_2.0x1.6mm
- moved R1 10.7 mm to (124.8, 104.6), turned to 90 degrees
- moved R6 9.94 mm to (123.8, 104.6), turned to 90 degrees
- moved R18 7.47 mm to (129.8, 114.9), turned to 315 degrees
- moved R5 6.84 mm to (129.6, 120.3), turned to 315 degrees
- moved R2 6.79 mm to (122.6, 114.6), turned to 315 degrees
- moved R4 5.52 mm to (129.0, 121.0), turned to 135 degrees
- moved R19 3.76 mm to (128.6, 113.8), turned to 315 degrees
- moved U1 3.40 mm to (127.1, 116.5), turned to 225 degrees
- moved C9 2.90 mm to (149.8, 96.6), turned to 270 degrees
- moved R3 2.44 mm to (123.3, 113.9), turned to 135 degrees
- moved C11 2.03 mm to (123.3, 97.1), turned to 180 degrees
- moved R11 1.97 mm to (123.3, 99.0), turned to 0 degrees
- moved M1 0.69 mm to (151.7, 96.6), turned to 270 degrees
- moved C10 0.64 mm to (123.3, 98.0), turned to 180 degrees
Connections:
- U1 pad 1: /USB_Connection/Switch -> /USB_Connection/CCV
- U1 pad 12: /USB_Connection/CCV -> /USB_Connection/CC2
- U1 pad 13: Net-(R4-Pad2) -> /USB_Connection/CC1
- U1 pad 14: /Bottom_Interface/3A_DET -> /USB_Connection/Switch
- U1 pad 2: /USB_Connection/CC1 -> /USB_Connection/CCV
- U1 pad 3: /USB_Connection/CC2 -> Net-(R18-Pad2)
- U1 pad 5: Net-(R18-Pad2) -> /USB_Connection/CCV
- U1 pad 6: /USB_Connection/CCV -> Net-(R2-Pad2)
- U1 pad 7: /USB_Connection/CCV -> /Bottom_Interface/1.5A_DET
- U1 pad 8: /Bottom_Interface/1.5A_DET -> /Bottom_Interface/3A_DET
- U1 pad 9: Net-(R2-Pad2) -> Net-(R4-Pad2)
- U2 pad A1: Net-(U2-PadA1) -> /ho
- U2 pad A2: Net-(U2-PadA2) -> /ho
Routing:
- net /USB_Connection/CCV: track 0.00 -> 10.3 mm
- net Net-(R18-Pad2): track 0.00 -> 9.26 mm
- net /USB_Connection/CC2: track 0.00 -> 4.61 mm
- net GND: track 88.0 -> 91.9 mm, vias 19 -> 20
- net /USB_Connection/CC1: track 0.00 -> 3.60 mm
- net Earth: track 0.00 -> 3.08 mm
