File: KiCad/Super_Blaster_v0.1.kicad_pcb (KiCad board)
At the start: 4 copper layers, 55 x 35 mm, 76 parts, among them J1 USB_TypeC_AMP_12401610E4#2A, J2 Conn_02x25_Odd_Even, J3 Conn_02x25_Odd_Even, M1 CLOCK_EN, U1 MCP6L94, U2 iCE40-HX8K-CT256, U3 FUSB340, U4 FT601Q, U5 REG_EN_GND_LX_VIN_NC_FB, U6 REG_EN_GND_LX_VIN_NC_FB, Y1 30MHz

Commit message: refreshing memory...
Parts:
- D1: footprint Diodes_SMD:D_SOD-323 -> Diode_SMD:D_0402_1005Metric
- R1, R6: moved to F.Cu
- moved R1 10.7 mm to (130.5, 113.8), turned to 45 degrees
- moved R6 10.3 mm to (129.8, 113.1), turned to 45 degrees
- moved D1 2.80 mm to (158.6, 107.3), turned to 135 degrees
- moved C20 0.60 mm to (160.6, 104.0)
- moved C30 0.52 mm to (158.0, 98.1)
- moved C17 0.32 mm to (158.5, 101.7)
- moved C33 0.22 mm to (156.4, 100.1)
- moved C24 0.17 mm to (161.2, 111.0)
- moved C43 0.16 mm to (160.4, 113.0)
- moved R10 0.15 mm to (139.9, 95.0)
- moved C35 0.13 mm to (158.9, 105.3)
- moved R17 0.12 mm to (160.9, 107.3)
- moved C6 0.12 mm to (136.8, 102.4)
- moved C39 0.11 mm to (161.5, 105.1)
- moved C7 0.09 mm to (138.7, 100.4)
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Routing:
- net 3v3: track 15.9 -> 119.1 mm, vias 14 -> 23
- net USB_V: track 5.77 -> 97.0 mm, vias 10 -> 13
- net VD10: track 4.05 -> 25.1 mm, vias 1 -> 4
- net /USB_Connection/CC1: track 3.60 -> 23.9 mm, vias 0 -> 2
- net /USB_Connection/CC2: track 4.61 -> 20.9 mm, vias 0 -> 2
- net Net-(J3-Pad21): track 0.00 -> 15.4 mm
- net Net-(J3-Pad33): track 0.00 -> 15.2 mm
- net Net-(U2-PadB12): track 19.9 -> 4.95 mm
- net Net-(U2-PadB14): track 17.5 -> 3.07 mm
- net Net-(J3-Pad19): track 0.00 -> 14.1 mm
- net Net-(J3-Pad31): track 0.00 -> 14.0 mm
- net Net-(U2-PadC12): track 3.45 -> 17.1 mm
- net Net-(J3-Pad17): track 0.00 -> 12.7 mm
- net Net-(J3-Pad29): track 0.00 -> 12.6 mm
- net /USB_Connection/Switch: track 0.00 -> 12.5 mm, vias 0 -> 2
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Other:
- net class 10 mil: clearance 0.1524 -> 0.127
- net class Default: clearance 0.1524 -> 0.10922
- rule pad_to_mask_clearance: 0.0762 -> 0.0381
- rule trace_clearance: 0.1524 -> 0.10922
- rule trace_min: 0.1016 -> 0.127
